File: hardware/X100_V1/02_MCU.kicad_sch (KiCad schematic)
At the start: 33 parts, among them U201 STM32H743VIT6, Y201 8.000MHz /CL20pF

Commit message: Refactor X100 schematics for readability
Other:
- note added: "02 主控与时钟 / MCU AND CLOCK"
- note added: "BOOT0 默认LOW · 恢复方式见页底说明"
- note added: "HSE 晶振 / HSE CLOCK · 8.000 MHz"
- note added: "POWER / CONTROL"
- note added: "PWM / ADC"
- note added: "SDMMC"
- note added: "SPI / IMU / BARO"
- note added: "STM32H743 主控与去耦 / MCU CORE AND DECOUPLING"
- note added: "UART / I2C"
- note added: "USB / CAN / DEBUG"
- note added: "VCAP 核心稳压 / CORE REGULATOR"
- note added: "VDD 去耦 / VDD DECOUPLING"
- note added: "启动配置 / BOOT CONFIGURATION"
- note added: "复位 / RESET"
- note added: "模拟与备份供电 / ANALOG AND BACKUP POWER"
- note added: "状态与电源指示 / STATUS AND PWR LED"
- moved on the sheet: C201, C202, C203, C204, C205, C206, C207, C208, C209, C210, C211, C212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

Commit message: 紧凑测试点保留65处可测性并消除46对courtyard重叠
Parts:
- TP201, TP202, TP203, TP204, TP208: footprint X100_Physical:TP1p5_NoPaste -> X100_Physical:TP0p6_Inline_NoPaste; Layout Note (none) -> 0.6mm probe land, unchanged 0.5mm probe envelope; fine-tip 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; MPN TP1p5 -> PCB_TESTPAD_0P6_NO_PASTE; Package 1.5mm top probe -> PCB feature: 0.6mm exposed round test land; no paste
Changed lines of the file:
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@@
 			)
 		)
-		(property "Footprint" "X100_Physical:TP1p5_NoPaste"
+		(property "Footprint" "X100_Physical:TP0p6_Inline_NoPaste"
 			(at 406.4 308.61 0)
 			(effects
@@
 			)
 		)
-		(property "MPN" "TP1p5"
+		(property "MPN" "PCB_TESTPAD_0P6_NO_PASTE"
 			(at 406.4 308.61 0)
 			(effects
@@
 			)
 		)
-		(property "Package" "1.5mm top probe"
+		(property "Package" "PCB feature: 0.6mm exposed round test land; no paste"
 			(at 406.4 308.61 0)
 			(effects
@@
 			)
 		)
+    (property "Layout Note" "0.6mm probe land, unchanged 0.5mm probe envelope; fine-tip probing; all 65 net accesses retained" (at 406.4 308.61 0)
+      (effects (font (size 1.27 1.27)) (hide yes))
+    )
 		(instances
 			(project "X100_CleanSheet"
@@
 			)
 		)
-		(property "Footprint" "X100_Physical:TP1p5_NoPaste"
+		(property "Footprint" "X100_Physical:TP0p6_Inline_NoPaste"
 			(at 449.58 308.61 0)
 			(effects
@@
 			)
 		)
-		(property "MPN" "TP1p5"
+		(property "MPN" "PCB_TESTPAD_0P6_NO_PASTE"
 			(at 449.58 308.61 0)
 			(effects
@@
 			)
 		)
-		(property "Package" "1.5mm top probe"
+		(property "Package" "PCB feature: 0.6mm exposed round test land; no paste"
 			(at 449.58 308.61 0)
 			(effects
@@
 			)
 		)
+    (property "Layout Note" "0.6mm probe land, unchanged 0.5mm probe envelope; fine-tip probing; all 65 net accesses retained" (at 449.58 308.61 0)
+      (effects (font (size 1.27 1.27)) (hide yes))
+    )
 		(instances
 			(project "X100_CleanSheet"
@@
 			)
 		)
-		(property "Footprint" "X100_Physical:TP1p5_NoPaste"
+		(property "Footprint" "X100_Physical:TP0p6_Inline_NoPaste"
 			(at 492.76 308.61 0)
 			(effects
@@
 			)
 		)
-		(property "MPN" "TP1p5"
+		(property "MPN" "PCB_TESTPAD_0P6_NO_PASTE"
 			(at 492.76 308.61 0)
 			(effects
@@
 			)
 		)
-		(property "Package" "1.5mm top probe"
+		(property "Package" "PCB feature: 0.6mm exposed round test land; no paste"
 			(at 492.76 308.61 0)
 			(effects
@@
 			)
 		)
+    (property "Layout Note" "0.6mm probe land, unchanged 0.5mm probe envelope; fine-tip probing; all 65 net accesses retained" (at 492.76 308.61 0)
+      (effects (font (size 1.27 1.27)) (hide yes))
+    )
 		(instances
 			(project "X100_CleanSheet"
@@
 			)
 		)
-		(property "Footprint" "X100_Physical:TP1p5_NoPaste"
+		(property "Footprint" "X100_Physical:TP0p6_Inline_NoPaste"
 			(at 535.94 308.61 0)
 			(effects
@@
 			)
 		)
-		(property "MPN" "TP1p5"
+		(property "MPN" "PCB_TESTPAD_0P6_NO_PASTE"
 			(at 535.94 308.61 0)
 			(effects
@@
 			)
 		)
-		(property "Package" "1.5mm top probe"
+		(property "Package" "PCB feature: 0.6mm exposed round test land; no paste"
 			(at 535.94 308.61 0)
 			(effects
@@
 			)
 		)
+    (property "Layout Note" "0.6mm probe land, unchanged 0.5mm probe envelope; fine-tip probing; all 65 net accesses retained" (at 535.94 308.61 0)
+      (effects (font (size 1.27 1.27)) (hide yes))
+    )
 		(instances
 			(project "X100_CleanSheet"
@@
 			)
 		)
-		(property "Footprint" "X100_Physical:TP1p5_NoPaste"
+		(property "Footprint" "X100_Physical:TP0p6_Inline_NoPaste"
 			(at 535.94 322.58 0)
 			(effects
@@
 			)
 		)
-		(property "MPN" "TP1p5"
+		(property "MPN" "PCB_TESTPAD_0P6_NO_PASTE"
 			(at 535.94 322.58 0)
 			(effects
@@
 			)
 		)
-		(property "Package" "1.5mm top probe"
+		(property "Package" "PCB feature: 0.6mm exposed round test land; no paste"
 			(at 535.94 322.58 0)
 			(effects
@@
 			)
 		)
+    (property "Layout Note" "0.6mm probe land, unchanged 0.5mm probe envelope; fine-tip probing; all 65 net accesses retained" (at 535.94 322.58 0)
+      (effects (font (size 1.27 1.27)) (hide yes))
+    )
 		(instances
 			(project "X100_CleanSheet"
