File: hardware/X100_V1/05_SD.kicad_sch (KiCad schematic)
At the start: 17 parts, among them J501 1040310811

Commit message: Refactor X100 schematics for readability
Other:
- note added: "05 microSD数据存储 / MICROSD STORAGE"
- note added: "POWER / GND"
- note added: "SDMMC / SIGNALS"
- note added: "STM32 SDMMC1 ↔ microSD · 3.3V / 4-bit"
- note added: "microSD 接口与信号上拉 / MICROSD AND SDMMC PULLUPS"
- note added: "本地供电与去耦 / LOCAL POWER AND DECOUPLING"
- moved on the sheet: C501, C502, J501, R501, R502, R503, R504, R505, R506, TP501, TP502, TP503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

Commit message: 紧凑测试点保留65处可测性并消除46对courtyard重叠
Parts:
- TP501, TP508: footprint X100_Physical:TP1p5_NoPaste -> X100_Physical:TP0p6_Inline_NoPaste; Layout Note (none) -> 0.6mm probe land, unchanged 0.5mm probe envelope; fine-tip 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; MPN TP1p5 -> PCB_TESTPAD_0P6_NO_PASTE; Package 1.5mm top probe -> PCB feature: 0.6mm exposed round test land; no paste
Changed lines of the file:
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@@
 			)
 		)
-		(property "Footprint" "X100_Physical:TP1p5_NoPaste"
+		(property "Footprint" "X100_Physical:TP0p6_Inline_NoPaste"
 			(at 284.48 332.74 0)
 			(effects
@@
 			)
 		)
-		(property "MPN" "TP1p5"
+		(property "MPN" "PCB_TESTPAD_0P6_NO_PASTE"
 			(at 284.48 332.74 0)
 			(effects
@@
 			)
 		)
-		(property "Package" "1.5mm top probe"
+		(property "Package" "PCB feature: 0.6mm exposed round test land; no paste"
 			(at 284.48 332.74 0)
 			(effects
@@
 			)
 		)
+    (property "Layout Note" "0.6mm probe land, unchanged 0.5mm probe envelope; fine-tip probing; all 65 net accesses retained" (at 284.48 332.74 0)
+      (effects (font (size 1.27 1.27)) (hide yes))
+    )
 		(instances
 			(project "X100_CleanSheet"
@@
 			)
 		)
-		(property "Footprint" "X100_Physical:TP1p5_NoPaste"
+		(property "Footprint" "X100_Physical:TP0p6_Inline_NoPaste"
 			(at 497.84 360.68 0)
 			(effects
@@
 			)
 		)
-		(property "MPN" "TP1p5"
+		(property "MPN" "PCB_TESTPAD_0P6_NO_PASTE"
 			(at 497.84 360.68 0)
 			(effects
@@
 			)
 		)
-		(property "Package" "1.5mm top probe"
+		(property "Package" "PCB feature: 0.6mm exposed round test land; no paste"
 			(at 497.84 360.68 0)
 			(effects
@@
 			)
 		)
+    (property "Layout Note" "0.6mm probe land, unchanged 0.5mm probe envelope; fine-tip probing; all 65 net accesses retained" (at 497.84 360.68 0)
+      (effects (font (size 1.27 1.27)) (hide yes))
+    )
 		(instances
 			(project "X100_CleanSheet"
