File: hardware/X100_V1/06_CAN.kicad_sch (KiCad schematic)
At the start: 12 parts, among them J601 SM04B-GHS-TB(LF)(SN), U601 TCAN3414DR

Commit message: Refactor X100 schematics for readability
Other:
- note added: "06 CAN通信 / CAN INTERFACE"
- note added: "120Ω 终端 / CAN TERMINATION · 默认OPEN"
- note added: "CAN 总线接口 / CAN BUS CONNECTOR"
- note added: "CAN 收发器 / CAN TRANSCEIVER"
- note added: "CANH / CANL / POWER"
- note added: "CANH → R602 → CAN_TERM → JP601 → CANL"
- note added: "MCU / CONTROL"
- note added: "接口与测点 / INTERFACES AND TEST POINTS"
- moved on the sheet: C601, J601, JP601, R601, R602, R603, TP601, TP602, TP603, TP604, TP605, U601

Commit message: 紧凑测试点保留65处可测性并消除46对courtyard重叠
Parts:
- TP601, TP602, TP603, TP604, TP605: footprint X100_Physical:TP1p5_NoPaste -> X100_Physical:TP0p6_Inline_NoPaste; Layout Note (none) -> 0.6mm probe land, unchanged 0.5mm probe envelope; fine-tip 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; MPN TP1p5 -> PCB_TESTPAD_0P6_NO_PASTE; Package 1.5mm top probe -> PCB feature: 0.6mm exposed round test land; no paste
Changed lines of the file:
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@@
 			)
 		)
-		(property "Footprint" "X100_Physical:TP1p5_NoPaste"
+		(property "Footprint" "X100_Physical:TP0p6_Inline_NoPaste"
 			(at 284.48 283.21 0)
 			(effects
@@
 			)
 		)
-		(property "MPN" "TP1p5"
+		(property "MPN" "PCB_TESTPAD_0P6_NO_PASTE"
 			(at 284.48 283.21 0)
 			(effects
@@
 			)
 		)
-		(property "Package" "1.5mm top probe"
+		(property "Package" "PCB feature: 0.6mm exposed round test land; no paste"
 			(at 284.48 283.21 0)
 			(effects
@@
 			)
 		)
+    (property "Layout Note" "0.6mm probe land, unchanged 0.5mm probe envelope; fine-tip probing; all 65 net accesses retained" (at 284.48 283.21 0)
+      (effects (font (size 1.27 1.27)) (hide yes))
+    )
 		(instances
 			(project "X100_CleanSheet"
@@
 			)
 		)
-		(property "Footprint" "X100_Physical:TP1p5_NoPaste"
+		(property "Footprint" "X100_Physical:TP0p6_Inline_NoPaste"
 			(at 375.92 283.21 0)
 			(effects
@@
 			)
 		)
-		(property "MPN" "TP1p5"
+		(property "MPN" "PCB_TESTPAD_0P6_NO_PASTE"
 			(at 375.92 283.21 0)
 			(effects
@@
 			)
 		)
-		(property "Package" "1.5mm top probe"
+		(property "Package" "PCB feature: 0.6mm exposed round test land; no paste"
 			(at 375.92 283.21 0)
 			(effects
@@
 			)
 		)
+    (property "Layout Note" "0.6mm probe land, unchanged 0.5mm probe envelope; fine-tip probing; all 65 net accesses retained" (at 375.92 283.21 0)
+      (effects (font (size 1.27 1.27)) (hide yes))
+    )
 		(instances
 			(project "X100_CleanSheet"
@@
 			)
 		)
-		(property "Footprint" "X100_Physical:TP1p5_NoPaste"
+		(property "Footprint" "X100_Physical:TP0p6_Inline_NoPaste"
 			(at 467.36 283.21 0)
 			(effects
@@
 			)
 		)
-		(property "MPN" "TP1p5"
+		(property "MPN" "PCB_TESTPAD_0P6_NO_PASTE"
 			(at 467.36 283.21 0)
 			(effects
@@
 			)
 		)
-		(property "Package" "1.5mm top probe"
+		(property "Package" "PCB feature: 0.6mm exposed round test land; no paste"
 			(at 467.36 283.21 0)
 			(effects
@@
 			)
 		)
+    (property "Layout Note" "0.6mm probe land, unchanged 0.5mm probe envelope; fine-tip probing; all 65 net accesses retained" (at 467.36 283.21 0)
+      (effects (font (size 1.27 1.27)) (hide yes))
+    )
 		(instances
 			(project "X100_CleanSheet"
@@
 			)
 		)
-		(property "Footprint" "X100_Physical:TP1p5_NoPaste"
+		(property "Footprint" "X100_Physical:TP0p6_Inline_NoPaste"
 			(at 284.48 308.61 0)
 			(effects
@@
 			)
 		)
-		(property "MPN" "TP1p5"
+		(property "MPN" "PCB_TESTPAD_0P6_NO_PASTE"
 			(at 284.48 308.61 0)
 			(effects
@@
 			)
 		)
-		(property "Package" "1.5mm top probe"
+		(property "Package" "PCB feature: 0.6mm exposed round test land; no paste"
 			(at 284.48 308.61 0)
 			(effects
@@
 			)
 		)
+    (property "Layout Note" "0.6mm probe land, unchanged 0.5mm probe envelope; fine-tip probing; all 65 net accesses retained" (at 284.48 308.61 0)
+      (effects (font (size 1.27 1.27)) (hide yes))
+    )
 		(instances
 			(project "X100_CleanSheet"
@@
 			)
 		)
-		(property "Footprint" "X100_Physical:TP1p5_NoPaste"
+		(property "Footprint" "X100_Physical:TP0p6_Inline_NoPaste"
 			(at 375.92 308.61 0)
 			(effects
@@
 			)
 		)
-		(property "MPN" "TP1p5"
+		(property "MPN" "PCB_TESTPAD_0P6_NO_PASTE"
 			(at 375.92 308.61 0)
 			(effects
@@
 			)
 		)
-		(property "Package" "1.5mm top probe"
+		(property "Package" "PCB feature: 0.6mm exposed round test land; no paste"
 			(at 375.92 308.61 0)
 			(effects
@@
 			)
 		)
+    (property "Layout Note" "0.6mm probe land, unchanged 0.5mm probe envelope; fine-tip probing; all 65 net accesses retained" (at 375.92 308.61 0)
+      (effects (font (size 1.27 1.27)) (hide yes))
+    )
 		(instances
 			(project "X100_CleanSheet"
