File: hardware/X100_V1/01_POWER.kicad_sch (KiCad schematic)
At the start: 53 parts, among them Q101 DMP6023LSS-13, U101 TPS54360BDDAR, U102 AP63203WU-7, U103 TPS7A2033PDBVR, U104 TPS2553DBVR

Commit message: Refactor X100 schematics for readability
Other:
- note added: "01 电源管理 / POWER MANAGEMENT"
- note added: "BOOT / SW / EN / RT / FB / COMP — 原网络保持"
- note added: "EXTERNAL 5V / GND"
- note added: "MCU / SENSOR POWER"
- note added: "MCU 3.3V 电源 / MCU 3V3 SUPPLY"
- note added: "VBAT / MAIN 5V"
- note added: "VBAT 输入与保护 / VBAT INPUT AND PROTECTION"
- note added: "VBAT_RAW → VBAT_FUSED → VBAT_PROTECTED"
- note added: "主 5V 降压电源 / MAIN 5V BUCK"
- note added: "传感器 3.3V 电源 / SENSOR 3V3"
- note added: "受控外部 5V / CONTROLLED EXTERNAL 5V"
- moved on the sheet: C101, C102, C103, C104, C105, C106, C107, C108, C109, C110, C111, C112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

Commit message: 紧凑测试点保留65处可测性并消除46对courtyard重叠
Parts:
- TP101, TP106, TP107, TP108, TP109, TP110: footprint X100_Physical:TP1p5_NoPaste -> X100_Physical:TP0p6_Inline_NoPaste; Layout Note (none) -> 0.6mm probe land, unchanged 0.5mm probe envelope; fine-tip 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; MPN TP1p5 -> PCB_TESTPAD_0P6_NO_PASTE; Package 1.5mm top probe -> PCB feature: 0.6mm exposed round test land; no paste
Changed lines of the file:
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@@
 			)
 		)
-		(property "Footprint" "X100_Physical:TP1p5_NoPaste"
+		(property "Footprint" "X100_Physical:TP0p6_Inline_NoPaste"
 			(at 290.83 351.79 0)
 			(effects
@@
 			)
 		)
-		(property "MPN" "TP1p5"
+		(property "MPN" "PCB_TESTPAD_0P6_NO_PASTE"
 			(at 290.83 351.79 0)
 			(effects
@@
 			)
 		)
-		(property "Package" "1.5mm top probe"
+		(property "Package" "PCB feature: 0.6mm exposed round test land; no paste"
 			(at 290.83 351.79 0)
 			(effects
@@
 			)
 		)
+    (property "Layout Note" "0.6mm probe land, unchanged 0.5mm probe envelope; fine-tip probing; all 65 net accesses retained" (at 290.83 351.79 0)
+      (effects (font (size 1.27 1.27)) (hide yes))
+    )
 		(instances
 			(project "X100_CleanSheet"
@@
 			)
 		)
-		(property "Footprint" "X100_Physical:TP1p5_NoPaste"
+		(property "Footprint" "X100_Physical:TP0p6_Inline_NoPaste"
 			(at 360.68 365.76 0)
 			(effects
@@
 			)
 		)
-		(property "MPN" "TP1p5"
+		(property "MPN" "PCB_TESTPAD_0P6_NO_PASTE"
 			(at 360.68 365.76 0)
 			(effects
@@
 			)
 		)
-		(property "Package" "1.5mm top probe"
+		(property "Package" "PCB feature: 0.6mm exposed round test land; no paste"
 			(at 360.68 365.76 0)
 			(effects
@@
 			)
 		)
+    (property "Layout Note" "0.6mm probe land, unchanged 0.5mm probe envelope; fine-tip probing; all 65 net accesses retained" (at 360.68 365.76 0)
+      (effects (font (size 1.27 1.27)) (hide yes))
+    )
 		(instances
 			(project "X100_CleanSheet"
@@
 			)
 		)
-		(property "Footprint" "X100_Physical:TP1p5_NoPaste"
+		(property "Footprint" "X100_Physical:TP0p6_Inline_NoPaste"
 			(at 430.53 365.76 0)
 			(effects
@@
 			)
 		)
-		(property "MPN" "TP1p5"
+		(property "MPN" "PCB_TESTPAD_0P6_NO_PASTE"
 			(at 430.53 365.76 0)
 			(effects
@@
 			)
 		)
-		(property "Package" "1.5mm top probe"
+		(property "Package" "PCB feature: 0.6mm exposed round test land; no paste"
 			(at 430.53 365.76 0)
 			(effects
@@
 			)
 		)
+    (property "Layout Note" "0.6mm probe land, unchanged 0.5mm probe envelope; fine-tip probing; all 65 net accesses retained" (at 430.53 365.76 0)
+      (effects (font (size 1.27 1.27)) (hide yes))
+    )
 		(instances
 			(project "X100_CleanSheet"
@@
 			)
 		)
-		(property "Footprint" "X100_Physical:TP1p5_NoPaste"
+		(property "Footprint" "X100_Physical:TP0p6_Inline_NoPaste"
 			(at 500.38 365.76 0)
 			(effects
@@
 			)
 		)
-		(property "MPN" "TP1p5"
+		(property "MPN" "PCB_TESTPAD_0P6_NO_PASTE"
 			(at 500.38 365.76 0)
 			(effects
@@
 			)
 		)
-		(property "Package" "1.5mm top probe"
+		(property "Package" "PCB feature: 0.6mm exposed round test land; no paste"
 			(at 500.38 365.76 0)
 			(effects
@@
 			)
 		)
+    (property "Layout Note" "0.6mm probe land, unchanged 0.5mm probe envelope; fine-tip probing; all 65 net accesses retained" (at 500.38 365.76 0)
+      (effects (font (size 1.27 1.27)) (hide yes))
+    )
 		(instances
 			(project "X100_CleanSheet"
@@
 			)
 		)
-		(property "Footprint" "X100_Physical:TP1p5_NoPaste"
+		(property "Footprint" "X100_Physical:TP0p6_Inline_NoPaste"
 			(at 290.83 379.73 0)
 			(effects
@@
 			)
 		)
-		(property "MPN" "TP1p5"
+		(property "MPN" "PCB_TESTPAD_0P6_NO_PASTE"
 			(at 290.83 379.73 0)
 			(effects
@@
 			)
 		)
-		(property "Package" "1.5mm top probe"
+		(property "Package" "PCB feature: 0.6mm exposed round test land; no paste"
 			(at 290.83 379.73 0)
 			(effects
@@
 			)
 		)
+    (property "Layout Note" "0.6mm probe land, unchanged 0.5mm probe envelope; fine-tip probing; all 65 net accesses retained" (at 290.83 379.73 0)
+      (effects (font (size 1.27 1.27)) (hide yes))
+    )
 		(instances
 			(project "X100_CleanSheet"
@@
 			)
 		)
-		(property "Footprint" "X100_Physical:TP1p5_NoPaste"
+		(property "Footprint" "X100_Physical:TP0p6_Inline_NoPaste"
 			(at 360.68 379.73 0)
 			(effects
@@
 			)
 		)
-		(property "MPN" "TP1p5"
+		(property "MPN" "PCB_TESTPAD_0P6_NO_PASTE"
 			(at 360.68 379.73 0)
 			(effects
@@
 			)
 		)
-		(property "Package" "1.5mm top probe"
+		(property "Package" "PCB feature: 0.6mm exposed round test land; no paste"
 			(at 360.68 379.73 0)
 			(effects
@@
 			)
 		)
+    (property "Layout Note" "0.6mm probe land, unchanged 0.5mm probe envelope; fine-tip probing; all 65 net accesses retained" (at 360.68 379.73 0)
+      (effects (font (size 1.27 1.27)) (hide yes))
+    )
 		(instances
 			(project "X100_CleanSheet"

Commit message: Adopt approved L101 SRP1038A and review actual 5V load
Parts:
- L101: footprint X100_Physical:Bourns_SRP1265A -> X100_Physical:Bourns_SRP1038A_LeadFrame_NoVIP; symbol X100_Physical:SRP1265A_100M -> X100_LayoutECO:Bourns_SRP1038A_100M; DCR Max (none) -> 30mOhm @25C; Inductance (none) -> 10uH +/-20% @100kHz/1V; Irms (none) -> 7.5A; rated40C rise; application thermal test required; Isat (none) -> 12A @25C for20% L drop; not hot minimum guarantee; LCSC (none) -> C780184; MPN SRP1265A-100M -> SRP1038A-100M; Package 13.5x12.5x6.2 SMD -> Lead-frame SMD; case max11.5x10.3x4.0mm; Procurement Policy EXACT_MPN_FROZEN -> EXACT_MPN_FROZEN; USER_APPROVED_20261023; NO_PURCHASE; Verification Status (none) -> DATASHEET_AND_LAYOUT_VERIFIED; POWER_REVIEW_OPEN; NO_BENCH_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
