File: hardware/proposals/Y201_YXC_5032_NOT_APPROVED/project/02_MCU.kicad_sch (KiCad schematic)
At the start: 33 parts, among them U201 STM32H743VIT6, Y201 8MHz CL20pF YXC candidate

Commit message: 按原厂100ppm温漂更正R205候选并重算启动筛查
Parts:
- R205: TCR <=50ppm/C -> <=100ppm/C
Changed lines of the file:
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@@
 			)
 		)
-		(property "Datasheet" "https://www.yageogroup.com/component-documentation/download/specsheet/RC0805FR-07120RL"
+		(property "Datasheet" "https://www.yageogroup.com/component-documentation/download/specsheet/RC0805FR-07100RL"
 			(at 54.61 66.04 0)
 			(effects
@@
 			)
 		)
-    (property "TCR" "<=50ppm/C" (at 54.61 66.04 0)
+    (property "TCR" "<=100ppm/C" (at 54.61 66.04 0)
       (effects (font (size 1.27 1.27)) (hide yes))
     )
